File: hardware/PowerFEC.kicad_pcb (KiCad board)
At the start: 2 copper layers, 24 x 27.9 mm, 28 parts, among them J1 105444-0001, J2 B2B-XH-A, U1 PIC16F1455, U2 AP22652, U3 ZXCT1009, U4 MCP3422

Commit message: Fixed refdes
Parts:
- renumbered R9 to R10, R4 to R5, R5 to R7, R7 to R8, R8 to R9
Changed lines of the file:
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@@
 		(at 37.5 38.5 90)
 		(tags "RESC2013X70N")
-		(property "Reference" "R5"
+		(property "Reference" "R7"
 			(at 0 -1.6 90)
 			(layer "F.SilkS")
@@
 		(at 27.7 31.5 90)
 		(tags "RESC2013X70N")
-		(property "Reference" "R9"
+		(property "Reference" "R10"
 			(at 0 -1.6 90)
 			(layer "F.SilkS")
@@
 		(at 39.7 38.5 -90)
 		(tags "RESC2013X70N")
-		(property "Reference" "R4"
+		(property "Reference" "R5"
 			(at 0 -1.6 90)
 			(layer "F.SilkS")
@@
 		)
 		(property "Value" "1K"
-			(at 2.4 0 0)
+			(at 2.4 0 180)
 			(layer "F.SilkS")
 			(effects
@@
 		(at 42.2 28 90)
 		(tags "RESC2013X70N")
-		(property "Reference" "R8"
+		(property "Reference" "R9"
 			(at 0 1.6 90)
 			(layer "B.SilkS")
@@
 		(at 40.2 28 90)
 		(tags "RESC2013X70N")
-		(property "Reference" "R7"
+		(property "Reference" "R8"
 			(at 0 1.6 90)
 			(layer "B.SilkS")
